Commit message: Fix ARX R5A gripper integration
Signed-off-by: wee733 <wee733@users.noreply.github.com>

File: isaac_ros_manipulation_arx_r5a_robot_description/urdf/r5a.ros2_control.xacro (robot description, xacro)
@@ -12,8 +12,7 @@
                 <param name="gripper_feedback_max">5.0</param>
                 <param name="gripper_command_max">5.0</param>
+                <param name="gripper_merge_policy">1</param>
                 <param name="max_arm_command_velocity">1.0</param>
-                <param name="max_gripper_command_velocity">0.02</param>
                 <param name="max_arm_command_lead">0.10</param>
-                <param name="max_gripper_command_lead">0.005</param>
                 <param name="status_timeout_ms">250</param>
             </hardware>
@@ -68,5 +67,4 @@
             </joint>
             <joint name="joint8">
-                <command_interface name="position"/>
                 <state_interface name="position">
                   <param name="initial_value">${initial_positions['joint8']}</param>

File: isaac_ros_manipulation_arx_r5a_robot_description/urdf/r5a.urdf (robot description, URDF)
Before this commit: robot R5a, 9 links, 8 joints
Joints:
- joint joint8: mimic (none) -> joint=joint7

File: isaac_ros_manipulation_arx_r5a_robot_description/urdf/r5a_cumotion.urdf (robot description, URDF)
Before this commit: robot R5a, 9 links, 8 joints
Joints:
- joint joint8: mimic (none) -> joint=joint7
