Commit message: Fix ARX R5A joint2 zero-position tolerance

File: isaac_ros_manipulation_arx_r5a_robot_description/urdf/r5a.urdf (robot description, URDF)
Before this commit: robot R5a, 9 links, 8 joints
Joints:
- joint joint2: limit lower=0.0 upper=3.0 effort=100 velocity=1000 -> lower=-0.01 upper=3.0 effort=100 velocity=1000

File: isaac_ros_manipulation_arx_r5a_robot_description/urdf/r5a_cumotion.urdf (robot description, URDF)
Before this commit: robot R5a, 9 links, 8 joints
Joints:
- joint joint2: limit lower=0.0 upper=3.0 effort=100 velocity=1.0 -> lower=-0.01 upper=3.0 effort=100 velocity=1.0

Commit message: Prepare ARX adapter for manipulation overlay
Add grasp and attachment frames, split cuMotion server and MoveIt plugin ownership, and document the standalone full-workflow overlay.

Signed-off-by: wee733 <wee733@users.noreply.github.com>

File: isaac_ros_manipulation_arx_r5a_robot_description/urdf/r5a.urdf (robot description, URDF)
Before this commit: robot R5a, 9 links, 8 joints
Links:
- added link grasp_frame
Joints:
- added joint grasp_frame_joint: type fixed, parent link6, child grasp_frame, origin xyz=0.11 0 0 rpy=0 0 0

File: isaac_ros_manipulation_arx_r5a_robot_description/urdf/r5a_cumotion.urdf (robot description, URDF)
Before this commit: robot R5a, 9 links, 8 joints
Links:
- added link grasp_frame
Joints:
- added joint grasp_frame_joint: type fixed, parent link6, child grasp_frame, origin xyz=0.11 0 0 rpy=0 0 0
